Commit message: added urdf meshes

File: urdf/dragoon.xacro (robot description, xacro)
@@ -1,4 +1,5 @@
 <?xml version="1.0"?>
 <robot name="dragoon" xmlns:xacro="http://www.ros.org/wiki/xacro">
+	<xacro:include filename="$(find dragoon_simulation)/urdf/dragoon_macros.xacro"/>
 	<material name="orange">
 		<color rgba="1.0 0.42342 0.039215 1.0"/>
@@ -12,5 +13,5 @@
 		<inertial>
 			<mass value="3.59"/>
-			<origin rpy="0 0 0" xyz="0 0.08 0" />
+			<origin rpy="1.57079 0 0" xyz="0 0.0 0" />
 			<inertia ixx="0.05" iyy="0.04" izz="0.08" ixy="0" ixz="0" iyz="0" />
 		</inertial>
@@ -22,67 +23,19 @@
 		</collision>
 		<visual>
-			<origin rpy="0 0 0" xyz="0 0 0" />
+			<origin rpy="1.57079 0 3.14159" xyz="0 0 0" />
 			<geometry>
-				<box size="0.4 0.2 0.1"/>
+				<mesh filename="package://dragoon_simulation/urdf/meshes/dragoon_base_with_wheel_base.STL" scale="0.001 0.001 0.001"/>
 			</geometry>
 			<material name="orange"/>
 		</visual>
 	</link>
-	<link name="link_right_wheel">
-		<inertial>
-			<mass value="0.129"/>
-			<origin rpy="0 0 0" xyz="0 0 0.004"/>
-			<inertia ixx="0.0001" iyy="0.0001" izz="0.0001" ixy="0" ixz="0" iyz="0" />
-		</inertial>
-		<collision name="link_right_wheel_collision">
-			<origin rpy="0 0 0" xyz="0 0 0"/>
-			<geometry>
-				<cylinder length="0.04" radius="0.1"/>
-			</geometry>
-		</collision>
-		<visual name="link_right_wheel_visual">
-			<origin rpy="0 0 0" xyz="0 0 0" />
-			<geometry>
-				<cylinder length="0.04" radius="0.1"/>
-			</geometry>
-			<material name="black"/>
-		</visual>
-	</link>
-	<joint name="joint_right_wheel" type="continuous">
-		<origin rpy="0 0 0" xyz="0 -0.5 0"/>
-		<child link="link_right_wheel"/>
-		<parent link="link_chassis"/>
-		<axis rpy=" 0 0 0" xyz="0 1 0"/>
-		<limit effort="10000" velocity="1000"/>
-		<joint_properties damping="1.0" friction="1.0"/>
-	</joint>
-	<link name="link_left_wheel">
-		<inertial>
-			<mass value="0.129"/>
-			<origin rpy="0 0 0" xyz="0 0 0.004"/>
-			<inertia ixx="0.0001" iyy="0.0001" izz="0.0001" ixy="0" ixz="0" iyz="0" />
-		</inertial>
-		<collision name="link_left_wheel_collision">
-			<origin rpy="0 0 0" xyz="0 0 0"/>
-			<geometry>
-				<cylinder length="0.04" radius="0.1"/>
-			</geometry>
-		</collision>
-		<visual name="link_left_wheel_visual">
-			<origin rpy="0 0 0" xyz="0 0 0" />
-			<geometry>
-				<cylinder length="0.04" radius="0.1"/>
-			</geometry>
-			<material name="black"/>
-		</visual>
-	</link>
-	<joint name="joint_left_wheel" type="continuous">
-		<origin rpy="0 0 0" xyz="0 0.5 0"/>
-		<child link="link_left_wheel"/>
-		<parent link="link_chassis"/>
-		<axis rpy=" 0 0 0" xyz="0 1 0"/>
-		<limit effort="10000" velocity="1000"/>
-		<joint_properties damping="1.0" friction="1.0"/>
-	</joint>
+	<xacro:wheel_link name="wheel_1_RF" origin_rpy="1.57079 0 0" origin_xyz="0 0 0"/>
+	<xacro:wheel_joint child="wheel_1_RF" parent="link_chassis" origin_xyz="0.1397 0.12764 0.02604" origin_rpy="0 0 0" />
+	<xacro:wheel_link name="wheel_2_LF" origin_rpy="1.57079 0 0" origin_xyz="0 0 0"/>
+	<xacro:wheel_joint child="wheel_2_LF" parent="link_chassis" origin_xyz="0.1397 -0.12764 0.02604" origin_rpy="0 0 0" />
+	<xacro:wheel_link name="wheel_3_RB" origin_rpy="1.57079 0 0" origin_xyz="0 0 0"/>
+	<xacro:wheel_joint child="wheel_3_RB" parent="link_chassis" origin_xyz="-0.1397 0.12764 0.02604" origin_rpy="0 0 0" />
+	<xacro:wheel_link name="wheel_4_LB" origin_rpy="1.57079 0 0" origin_xyz="0 0 0"/>
+	<xacro:wheel_joint child="wheel_4_LB" parent="link_chassis" origin_xyz="-0.1397 -0.12764 0.02604" origin_rpy="0 0 0" />
 	<gazebo>
 		<plugin name="gazebo_ros_control" filename="libgazebo_ros_control.so">

Commit message: updated meshes to be in full color, joints correct

File: urdf/dragoon.xacro (robot description, xacro)
@@ -13,5 +13,5 @@
 		<inertial>
 			<mass value="3.59"/>
-			<origin rpy="1.57079 0 0" xyz="0 0.0 0" />
+			<origin rpy="0 0 0" xyz="0 0.0 0" />
 			<inertia ixx="0.05" iyy="0.04" izz="0.08" ixy="0" ixz="0" iyz="0" />
 		</inertial>
@@ -19,22 +19,22 @@
 		<collision name="link_chassis_collision" >
 			<geometry>
-				<box size="0.4 0.2 0.1" />
+				<mesh filename="package://dragoon_simulation/urdf/meshes/dragoon_base.dae" scale="1 1 1"/>
 			</geometry>
 		</collision>
 		<visual>
-			<origin rpy="1.57079 0 3.14159" xyz="0 0 0" />
+			<origin rpy="0 0 0" xyz="0 0 0" />
 			<geometry>
-				<mesh filename="package://dragoon_simulation/urdf/meshes/dragoon_base_with_wheel_base.STL" scale="0.001 0.001 0.001"/>
+				<mesh filename="package://dragoon_simulation/urdf/meshes/dragoon_base.dae" scale="1 1 1"/>
 			</geometry>
 			<material name="orange"/>
 		</visual>
 	</link>
-	<xacro:wheel_link name="wheel_1_RF" origin_rpy="1.57079 0 0" origin_xyz="0 0 0"/>
+	<xacro:wheel_link name="wheel_1_RF" origin_rpy="0 0 0" origin_xyz="0 0 0"/>
 	<xacro:wheel_joint child="wheel_1_RF" parent="link_chassis" origin_xyz="0.1397 0.12764 0.02604" origin_rpy="0 0 0" />
-	<xacro:wheel_link name="wheel_2_LF" origin_rpy="1.57079 0 0" origin_xyz="0 0 0"/>
+	<xacro:wheel_link name="wheel_2_LF" origin_rpy="0 0 0" origin_xyz="0 0 0"/>
 	<xacro:wheel_joint child="wheel_2_LF" parent="link_chassis" origin_xyz="0.1397 -0.12764 0.02604" origin_rpy="0 0 0" />
-	<xacro:wheel_link name="wheel_3_RB" origin_rpy="1.57079 0 0" origin_xyz="0 0 0"/>
+	<xacro:wheel_link name="wheel_3_RB" origin_rpy="0 0 0" origin_xyz="0 0 0"/>
 	<xacro:wheel_joint child="wheel_3_RB" parent="link_chassis" origin_xyz="-0.1397 0.12764 0.02604" origin_rpy="0 0 0" />
-	<xacro:wheel_link name="wheel_4_LB" origin_rpy="1.57079 0 0" origin_xyz="0 0 0"/>
+	<xacro:wheel_link name="wheel_4_LB" origin_rpy="0 0 0" origin_xyz="0 0 0"/>
 	<xacro:wheel_joint child="wheel_4_LB" parent="link_chassis" origin_xyz="-0.1397 -0.12764 0.02604" origin_rpy="0 0 0" />
 	<gazebo>

File: urdf/dragoon_macros.xacro (robot description, xacro)
@@ -11,5 +11,5 @@
                 <origin rpy="${origin_rpy}" xyz="${origin_xyz}"/>
                 <geometry>
-                    <mesh filename="package://dragoon_simulation/urdf/meshes/wheel.STL" scale="0.001 0.001 0.001"/>
+                    <mesh filename="package://dragoon_simulation/urdf/meshes/wheel.STL" scale="1 1 1"/>
                 </geometry>
             </collision>
@@ -17,7 +17,6 @@
                 <origin rpy="${origin_rpy}" xyz="${origin_xyz}" />
                 <geometry>
-                    <mesh filename="package://dragoon_simulation/urdf/meshes/wheel.STL" scale="0.001 0.001 0.001"/>
+                    <mesh filename="package://dragoon_simulation/urdf/meshes/wheel.dae" scale="1 1 1"/>
                 </geometry>
-                <material name="black"/>
             </visual>
         </link>

Commit message: finally got gazebo model to work what a drag

File: urdf/dragoon.xacro (robot description, xacro)
@@ -19,5 +19,5 @@
 		<collision name="link_chassis_collision" >
 			<geometry>
-				<mesh filename="package://dragoon_simulation/urdf/meshes/dragoon_base.dae" scale="1 1 1"/>
+				<mesh filename="package://dragoon_simulation/meshes/dragoon_base.dae" scale="1 1 1"/>
 			</geometry>
 		</collision>
@@ -25,5 +25,5 @@
 			<origin rpy="0 0 0" xyz="0 0 0" />
 			<geometry>
-				<mesh filename="package://dragoon_simulation/urdf/meshes/dragoon_base.dae" scale="1 1 1"/>
+				<mesh filename="package://dragoon_simulation/meshes/dragoon_base.dae" scale="1 1 1"/>
 			</geometry>
 			<material name="orange"/>

File: urdf/dragoon_macros.xacro (robot description, xacro)
@@ -11,5 +11,5 @@
                 <origin rpy="${origin_rpy}" xyz="${origin_xyz}"/>
                 <geometry>
-                    <mesh filename="package://dragoon_simulation/urdf/meshes/wheel.STL" scale="1 1 1"/>
+                    <mesh filename="package://dragoon_simulation/meshes/wheel.dae" scale="1 1 1"/>
                 </geometry>
             </collision>
@@ -17,5 +17,5 @@
                 <origin rpy="${origin_rpy}" xyz="${origin_xyz}" />
                 <geometry>
-                    <mesh filename="package://dragoon_simulation/urdf/meshes/wheel.dae" scale="1 1 1"/>
+                    <mesh filename="package://dragoon_simulation/meshes/wheel.dae" scale="1 1 1"/>
                 </geometry>
             </visual>
